File: pcb/lisn-pcb/lisn_choke.sch (KiCad schematic (older format))
At the start: 11 parts

Commit message: finished PCB routing
Parts:
- L5: value 6.8u -> 10u; MPN 7443330680 -> 7443331000
- L6: value 3.3u -> 10u; MPN 7443340330 -> 7443331000
Changed lines of the file:
@@
 $Descr A4 11693 8268
 encoding utf-8
-Sheet 5 5
+Sheet 3 5
 Title ""
 Date ""
@@
 AR Path="/61009C0D/60FEB02E" Ref="L11"  Part="1"
 F 0 "L11" H 6250 2215 50  0000 C CNN
-F 1 "6.8u" H 6250 2124 50  0000 C CNN
+F 1 "10u" H 6250 2124 50  0000 C CNN
 F 2 "wbraun_smd:L_WURTH_WE-HCC-1090" H 6250 2000 50  0001 C CNN
 F 3 "~" H 6250 2000 50  0001 C CNN
-F 4 "7443330680" H 6250 2000 50  0001 C CNN "MPN"
+F 4 "7443331000" H 6250 2000 50  0001 C CNN "MPN"
 	1    6250 2000
 	1    0    0    -1
@@
 AR Path="/61009C0D/60FEB268" Ref="L12"  Part="1"
 F 0 "L12" H 7250 2215 50  0000 C CNN
-F 1 "3.3u" H 7250 2124 50  0000 C CNN
+F 1 "10u" H 7250 2124 50  0000 C CNN
 F 2 "wbraun_smd:L_WURTH_WE-HCC-1090" H 7250 2000 50  0001 C CNN
 F 3 "~" H 7250 2000 50  0001 C CNN
-F 4 "7443340330" H 7250 2000 50  0001 C CNN "MPN"
+F 4 "7443331000" H 7250 2000 50  0001 C CNN "MPN"
 	1    7250 2000
 	1    0    0    -1
