File: pcb/lisn-pcb/lisn-pcb.kicad_pcb (KiCad board)
At the start: 2 copper layers, 160 x 159 mm, 81 parts, among them J1 Conn_Coaxial, J2 Conn_Coaxial, J3 62409-1, J4 62409-1, J5 62409-1, J6 62409-1, J7 62409-1, J8 62409-1

Commit message: finished PCB routing
Parts:
- added G***: LOGO, wbraun_smd:bee_large_v3, F.Cu at (149.0, 57.0)
- added H1: MountingHole_Pad, wbraun_smd:M3-tight-fit-socket-head, F.Cu at (255.2, 195.2)
- added H2: MountingHole_Pad, wbraun_smd:M3-tight-fit-socket-head, F.Cu at (104.8, 45.8)
- added H3: MountingHole_Pad, wbraun_smd:M3-tight-fit-socket-head, F.Cu at (104.8, 195.2)
- added H4: MountingHole_Pad, wbraun_smd:M3-tight-fit-socket-head, F.Cu at (255.2, 45.8)
- added J9: 62409-1, wbraun_smd:62409-1, F.Cu at (216.5, 185.0)
- added REF**: Symbol_Highvoltage_Type2_CopperTop_Small, Symbol:Symbol_Highvoltage_Type2_CopperTop_Small, F.Cu at (122.2, 182.8)
- L11, L5: value 6.8u -> 10u
- L12, L6: value 3.3u -> 10u
- moved C2 27.5 mm to (117.0, 124.5), turned to 270 degrees
- moved GD1 13.0 mm to (159.5, 155.0), turned to 180 degrees
- moved TR1 10.6 mm to (187.8, 171.2)
- moved R5 8.00 mm to (187.5, 179.2), turned to 0 degrees
- moved R8 8.00 mm to (187.5, 185.2), turned to 0 degrees
- moved R3 7.22 mm to (194.5, 179.2), turned to 180 degrees
- moved R6 7.22 mm to (194.5, 185.2), turned to 180 degrees
- moved R7 5.85 mm to (186.2, 182.2)
- moved C12 5.76 mm to (224.5, 168.2)
- moved R4 5.30 mm to (195.5, 182.2), turned to 270 degrees
- moved GD2 4.28 mm to (200.5, 155.0)
- moved D2 3.81 mm to (162.5, 106.8)
- moved C7 3.20 mm to (164.5, 134.0)
- moved C8 3.20 mm to (164.5, 126.0)
- moved D1 3.20 mm to (166.8, 113.2)
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Connections:
- TR1 pad 4: /SIG1_LIM -> /SIG2_LIM
- TR1 pad 6: /SIG2_LIM -> /SIG1_LIM
Routing:
- net /SIG1_LIM: track 0.00 -> 94.1 mm
- net Net-(C4-Pad1): track 0.00 -> 92.1 mm
- net /SIG2_LIM: track 0.00 -> 90.1 mm
- net Net-(C1-Pad1): track 0.00 -> 73.0 mm
- net /SIG1: track 0.00 -> 28.2 mm
- net /SIG2: track 0.00 -> 25.7 mm
- net Net-(R3-Pad1): track 0.00 -> 21.6 mm
- net /LINE: track 0.00 -> 21.1 mm
- net /NEUTRAL: track 0.00 -> 20.3 mm
- net Net-(L8-Pad2): track 0.00 -> 18.6 mm
- net Net-(L5-Pad2): track 0.00 -> 18.6 mm
- net Net-(L4-Pad2): track 0.00 -> 18.6 mm
- net Net-(L3-Pad2): track 0.00 -> 18.6 mm
- net Net-(L2-Pad2): track 0.00 -> 18.6 mm
- net Net-(L11-Pad2): track 0.00 -> 18.6 mm
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- added copper zone on F.Cu, net /DUT_LINE
- added copper zone on F.Cu, net /DUT_NUT
- added copper zone on F.Cu, net /LINE
- added copper zone on F.Cu, net /NEUTRAL
- added copper zone on F.Cu, net /SIG1_LIM
- added copper zone on B.Cu, net GND
- added copper zone on F.Cu, net Net-(L10-Pad1)
- added copper zone on F.Cu, net Net-(L10-Pad2)
- added copper zone on F.Cu, net Net-(L11-Pad2)
- added copper zone on F.Cu, net Net-(L2-Pad2)
- added copper zone on F.Cu, net Net-(L3-Pad2)
- added copper zone on F.Cu, net Net-(L4-Pad2)
- added copper zone on F.Cu, net Net-(L5-Pad2)
- added copper zone on F.Cu, net Net-(L8-Pad2)
Other:
- board text added: "Beefield Labs 50uH AC LISN github.com/westonb/leery-lisn"
- board text added: "CM Output"
- board text added: "DM Output"
- board text added: "G N"
- board text added: "L G"
- board text added: "L G N"

Commit message: V1 pcb design finished
Parts:
- removed the G*** at (149.0, 57.0)
- added G***: LOGO, wbraun_smd:Beefield_logo, F.Cu at (147.2, 58.5)
- TR1: value ADT2-71T -> ADT2-71T+
