File: pcb/lisn-pcb/lisn-pcb.sch (KiCad schematic (older format))
At the start: 23 parts, among them J1 Conn_Coaxial, J2 Conn_Coaxial, J3 62409-1, J4 62409-1, J5 62409-1, J6 62409-1, J7 62409-1, J8 62409-1

Commit message: finished PCB routing
Parts:
- added H1, H2, H3, H4: MountingHole_Pad, wbraun_smd:M3-tight-fit-socket-head, symbol Mechanical:MountingHole_Pad
- added J9: 62409-1, wbraun_smd:62409-1, symbol Connector:Conn_01x01_Male
Connections:
- net GND: now also H1.1, H2.1, H3.1, H4.1, J9.1 (Pin_1)
- net SIG1_LIM: now also TR1.6; no longer TR1.4
- net SIG2_LIM: now also TR1.4; no longer TR1.6
Changed lines of the file:
@@
 Wire Wire Line
 	8750 5200 8750 5300
+Text Label 6100 4100 2    50   ~ 0
+SIG1_LIM
 Text Label 6100 3700 2    50   ~ 0
-SIG1_LIM
-Text Label 6100 4100 2    50   ~ 0
 SIG2_LIM
 Wire Wire Line
@@
 L power:GND #PWR0133
 U 1 1 610488B7
-P 10650 1800
-F 0 "#PWR0133" H 10650 1550 50  0001 C CNN
-F 1 "GND" H 10655 1627 50  0000 C CNN
-F 2 "" H 10650 1800 50  0001 C CNN
-F 3 "" H 10650 1800 50  0001 C CNN
-	1    10650 1800
+P 10650 2100
+F 0 "#PWR0133" H 10650 1850 50  0001 C CNN
+F 1 "GND" H 10655 1927 50  0000 C CNN
+F 2 "" H 10650 2100 50  0001 C CNN
+F 3 "" H 10650 2100 50  0001 C CNN
+	1    10650 2100
 	1    0    0    -1
 $EndComp
@@
 Wire Wire Line
 	10500 1700 10650 1700
-Wire Wire Line
-	10650 1700 10650 1800
+$Comp
+L Connector:Conn_01x01_Male J9
+U 1 1 6117D612
+P 10300 1950
+F 0 "J9" H 10408 2131 50  0000 C CNN
+F 1 "62409-1" H 10408 2040 50  0000 C CNN
+F 2 "wbraun_smd:62409-1" H 10300 1950 50  0001 C CNN
+F 3 "~" H 10300 1950 50  0001 C CNN
+F 4 "62409-1" H 10300 1950 50  0001 C CNN "MPN"
+	1    10300 1950
+	1    0    0    -1
+$EndComp
+Wire Wire Line
+	10500 1950 10650 1950
+Wire Wire Line
+	10650 1700 10650 1950
+Wire Wire Line
+	10650 1950 10650 2100
+Connection ~ 10650 1950
+$Comp
+L Mechanical:MountingHole_Pad H1
+U 1 1 611A79AF
+P 4350 5650
+F 0 "H1" H 4450 5699 50  0000 L CNN
+F 1 "MountingHole_Pad" H 4450 5608 50  0000 L CNN
+F 2 "wbraun_smd:M3-tight-fit-socket-head" H 4350 5650 50  0001 C CNN
+F 3 "~" H 4350 5650 50  0001 C CNN
+	1    4350 5650
+	1    0    0    -1
+$EndComp
+$Comp
+L Mechanical:MountingHole_Pad H2
+U 1 1 611A7CBD
+P 4350 6000
+F 0 "H2" H 4450 6049 50  0000 L CNN
+F 1 "MountingHole_Pad" H 4450 5958 50  0000 L CNN
+F 2 "wbraun_smd:M3-tight-fit-socket-head" H 4350 6000 50  0001 C CNN
+F 3 "~" H 4350 6000 50  0001 C CNN
+	1    4350 6000
+	1    0    0    -1
+$EndComp
+$Comp
+L Mechanical:MountingHole_Pad H3
+U 1 1 611A8393
+P 4350 6350
+F 0 "H3" H 4450 6399 50  0000 L CNN
+F 1 "MountingHole_Pad" H 4450 6308 50  0000 L CNN
+F 2 "wbraun_smd:M3-tight-fit-socket-head" H 4350 6350 50  0001 C CNN
+F 3 "~" H 4350 6350 50  0001 C CNN
+	1    4350 6350
+	1    0    0    -1
+$EndComp
+$Comp
+L Mechanical:MountingHole_Pad H4
+U 1 1 611A8616
+P 4350 6700
+F 0 "H4" H 4450 6749 50  0000 L CNN
+F 1 "MountingHole_Pad" H 4450 6658 50  0000 L CNN
+F 2 "wbraun_smd:M3-tight-fit-socket-head" H 4350 6700 50  0001 C CNN
+F 3 "~" H 4350 6700 50  0001 C CNN
+	1    4350 6700
+	1    0    0    -1
+$EndComp
+$Comp
+L power:GND #PWR0134
+U 1 1 611A88B0
+P 4050 7000
+F 0 "#PWR0134" H 4050 6750 50  0001 C CNN
+F 1 "GND" H 4055 6827 50  0000 C CNN
+F 2 "" H 4050 7000 50  0001 C CNN
+F 3 "" H 4050 7000 50  0001 C CNN
+	1    4050 7000
+	1    0    0    -1
+$EndComp
+Wire Wire Line
+	4350 6800 4050 6800
+Wire Wire Line
+	4050 6800 4050 7000
+Wire Wire Line
+	4350 6450 4050 6450
+Wire Wire Line
+	4050 6450 4050 6800
+Connection ~ 4050 6800
+Wire Wire Line
+	4350 6100 4050 6100
+Wire Wire Line
+	4050 6100 4050 6450
+Connection ~ 4050 6450
+Wire Wire Line
+	4350 5750 4050 5750
+Wire Wire Line
+	4050 5750 4050 6100
+Connection ~ 4050 6100
 $EndSCHEMATC

Commit message: V1 pcb design finished
Parts:
- R3: MPN (none) -> RNCP0805FTD49R9
- R4, R7: MPN (none) -> RC0805JR-070RL
- TR1: value ADT2-71T -> ADT2-71T+; MPN (none) -> ADT2-71T+
Changed lines of the file:
@@
 P 6350 3900
 F 0 "TR1" H 6350 4281 50  0000 C CNN
-F 1 "ADT2-71T" H 6350 4190 50  0000 C CNN
+F 1 "ADT2-71T+" H 6350 4190 50  0000 C CNN
 F 2 "RF_Mini-Circuits:Mini-Circuits_CD637_H5.23mm" H 6350 3550 50  0001 C CNN
 F 3 "https://www.minicircuits.com/pdfs/ADT2-71T+.pdf" H 6350 3900 50  0001 C CNN
+F 4 "ADT2-71T+" H 6350 3900 50  0001 C CNN "MPN"
 	1    6350 3900
 	-1   0    0    -1
@@
 F 2 "Resistor_SMD:R_0805_2012Metric" V 7830 3700 50  0001 C CNN
 F 3 "~" H 7900 3700 50  0001 C CNN
+F 4 "RC0805JR-070RL" H 7900 3700 50  0001 C CNN "MPN"
 	1    7900 3700
 	0    -1   -1   0
@@
 F 2 "Resistor_SMD:R_0805_2012Metric" V 6830 5300 50  0001 C CNN
 F 3 "~" H 6900 5300 50  0001 C CNN
+F 4 "RNCP0805FTD49R9" H 6900 5300 50  0001 C CNN "MPN"
 	1    6900 5300
 	1    0    0    -1
@@
 F 2 "Resistor_SMD:R_0805_2012Metric" V 7280 5000 50  0001 C CNN
 F 3 "~" H 7350 5000 50  0001 C CNN
+F 4 "RC0805JR-070RL" H 7350 5000 50  0001 C CNN "MPN"
 	1    7350 5000
 	0    -1   -1   0
